File: discipline-pcb.kicad_pcb (KiCad board)
At the start: 2 copper layers, 304.9 x 122.8 mm, 197 parts, among them J1 AVR-ISP-6, SW1 KEYSW, SW10 KEYSW, SW11 KEYSW, SW12 KEYSW, SW13 KEYSW, SW14 KEYSW, SW15 KEYSW, SW16 KEYSW, SW17 KEYSW, SW18 KEYSW, SW19 KEYSW, SW2 KEYSW, SW20 KEYSW, SW21 KEYSW, SW22 KEYSW, SW23 KEYSW, SW24 KEYSW, SW25 KEYSW, SW26 KEYSW, SW27 KEYSW, SW28 KEYSW, SW29 KEYSW, SW3 KEYSW, SW30 KEYSW, SW31 KEYSW, SW32 KEYSW, SW33 KEYSW, SW34 KEYSW, SW35 KEYSW, SW36 KEYSW, SW37 KEYSW, SW38 KEYSW, SW39 KEYSW, SW4 KEYSW, SW40 KEYSW, SW41 KEYSW, SW42 KEYSW, SW43 KEYSW, SW44 KEYSW, SW45 KEYSW, SW46 KEYSW, SW47 KEYSW, SW48 KEYSW, SW49 KEYSW, SW5 KEYSW, SW50 KEYSW, SW51 KEYSW, SW52 KEYSW, SW53 KEYSW, SW54 KEYSW, SW55 KEYSW, SW56 KEYSW, SW57 KEYSW, SW58 KEYSW, SW59 KEYSW, SW6 KEYSW, SW60 KEYSW, SW61 KEYSW, SW62 KEYSW, SW63 KEYSW, SW64 KEYSW, SW65 KEYSW, SW66 KEYSW, SW67 KEYSW, SW68 KEYSW, SW69 KEYSW, SW7 KEYSW, SW70 KEYSW, SW71 KEYSW, SW72 KEYSW, SW73 KEYSW, SW74 KEYSW, SW75 KEYSW, SW76 KEYSW, SW77 KEYSW, SW78 KEYSW, SW8 KEYSW, SW9 KEYSW, U1 ATmega32A-PU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

Commit message: ISO Only Remove all keyswitch for ANSI layout from the PCB (schematic not modified)
Parts:
- removed SW29: KEYSW, cftkb:SW_Cherry_MX1A_1.50u_PCBNOSCREEN
- removed SW43, SW45: KEYSW, cftkb:SW_Cherry_MX1A_2.25u_PCBNOSCREEN
Routing:
- net Net-(D57-Pad2): track 152.2 -> 171.9 mm
- net col13: track 161.3 -> 176.3 mm
- net col0: track 364.4 -> 352.1 mm
- net Net-(D64-Pad2): track 188.7 -> 186.9 mm
- net Net-(D43-Pad2): track 153.6 -> 152.5 mm
- net Net-(D29-Pad2): track 127.9 -> 127.0 mm
Other:
- board text removed: "2.25U ANSI"
- board text removed: "ANSI ENTER"

Commit message: Modify all PCB to match the ISO Only layout
Routing:
- net GND: vias 48 -> 49
Other:
- board text added: "7/2/2019 - updated 7/14/2020"
- board text added: "ISO Only"
- board text removed: "7/2/2019 - updated 12/3/2019"
