File: plate/discipline-pcb.kicad_pcb (KiCad board)
At the start: 2 copper layers, 305.8 x 96.2 mm, 3 parts

Commit message: Modify all PCB to match the ISO Only layout
Other:
- outline, holes or cut-outs redrawn
- board text added: "7/2/2019 - updated 7/14/2020"
- board text removed: "7/2/2019 - updated 12/3/2019"
